File: Hardware/Kicad/PL_Toon.kicad_pcb (KiCad board)
At the start: 2 copper layers, 90 x 102 mm, 39 parts, among them IC1 LD1117S50TR, J1 Conn_01x06, J10 Conn_01x02, J2 Conn_01x02, J3 Conn_01x01_Pin, J4 Conn_01x03, J5 Conn_01x05, J6 Conn_01x02, J7 Conn_01x05, J8 Conn_01x04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

Commit message: Update the PCB files
- Updated the files, to take into account small changes like Do Not Populate, and add resistors values to 330 Ohm in the case of the LED resistors.
- Added Bill Of Material
Parts:
- R1, R6: value ~ -> 330
