File: Hardware/Kicad/PL_Toon.kicad_sch (KiCad schematic)
At the start: 39 parts, among them IC1 LD1117S50TR, J1 Conn_01x06, J10 Conn_01x02, J2 Conn_01x02, J3 Conn_01x01_Pin, J4 Conn_01x03, J5 Conn_01x05, J6 Conn_01x02, J7 Conn_01x05, J8 Conn_01x04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

Commit message: Update the PCB files
- Updated the files, to take into account small changes like Do Not Populate, and add resistors values to 330 Ohm in the case of the LED resistors.
- Added Bill Of Material
Parts:
- D1: Aliexpress https://es.aliexpress.com/item/1005005641884699.html?spm=a2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 -> https://es.aliexpress.com/item/1005006127128914.html?spm=a2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
- J9: now not fitted
- LED1, LED2: Aliexpress (none) -> https://es.aliexpress.com/item/1005003446964388.html?spm=a2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
- R1, R6: value ~ -> 330
- SW1: Aliexpress (none) -> https://es.aliexpress.com/item/4001202080623.html?spm=a2g0o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
- U2: Aliexpress (none) -> https://es.aliexpress.com/item/1005006537133858.html?spm=a2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
- U4: value ROB-14450 -> TB6612FNG; Aliexpress (none) -> https://es.aliexpress.com/item/1005006246388728.html?spm=a2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; Check_prices https://www.snapeda.com/parts/ROB-14450/SparkFun+Electronic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 -> (none)
